File: KiCAD/CIB - Blanket Octopus.kicad_pcb (KiCad board)
At the start: 2 copper layers, 73 x 55.9 mm, 30 parts, among them J1 DA15, J2 DA15, J3 Pins 01-06, J4 Pins 07-09 + sheild, J6 Pin Header, J8 Pin Header

Commit message: .
Other:
- board text removed: "https://chargepoint.atlassian.net/wiki/spaces/EN/pages/4961604878/DAQ970A+breakout+boards"
